Commit message: complete twice car scheduler

File: src/agv_description/urdf/agv_robot.urdf.xacro (robot description, xacro)
@@ -1,5 +1,10 @@
 <?xml version="1.0"?>
 <robot name="agv_robot" xmlns:xacro="http://www.ros.org/wiki/xacro">
+  <xacro:arg name="namespace" default="agv"/>
+  <xacro:arg name="prefix" default=""/>
+  <xacro:arg name="enable_ros2_control" default="true"/>
   <xacro:property name="PI" value="3.14159265"/>
+  <xacro:property name="robot_namespace" value="$(arg namespace)"/>
+  <xacro:property name="prefix" value="$(arg prefix)"/>
   <xacro:property name="base_x"       value="0.65"/>
   <xacro:property name="base_y"       value="0.50"/>
@@ -12,13 +17,13 @@
   <material name="agv_grey">  <color rgba="0.5 0.5 0.5 1.0"/></material>
   <material name="agv_yellow"><color rgba="1.0 0.8 0.0 1.0"/></material>
-  <link name="base_footprint">
+  <link name="${prefix}base_footprint">
     <visual><geometry><sphere radius="0.001"/></geometry></visual>
   </link>
-  <joint name="base_footprint_joint" type="fixed">
-    <parent link="base_footprint"/>
-    <child  link="base_link"/>
+  <joint name="${prefix}base_footprint_joint" type="fixed">
+    <parent link="${prefix}base_footprint"/>
+    <child  link="${prefix}base_link"/>
     <origin xyz="0 0 ${wheel_r}" rpy="0 0 0"/>
   </joint>
-  <link name="base_link">
+  <link name="${prefix}base_link">
     <visual>
       <geometry><box size="${base_x} ${base_y} ${base_z}"/></geometry>
@@ -33,16 +38,16 @@
     </inertial>
   </link>
-  <gazebo reference="base_link">
+  <gazebo reference="${prefix}base_link">
     <material>Gazebo/Black</material>
   </gazebo>
   <xacro:macro name="wheel" params="name px py">
-    <joint name="${name}_joint" type="continuous">
-      <parent link="base_link"/>
-      <child  link="${name}_link"/>
+    <joint name="${prefix}${name}_joint" type="continuous">
+      <parent link="${prefix}base_link"/>
+      <child  link="${prefix}${name}_link"/>
       <origin xyz="${px} ${py} ${-base_z/2}" rpy="${-PI/2} 0 0"/>
       <axis xyz="0 0 1"/>
       <dynamics damping="0.1" friction="0.5"/>
     </joint>
-    <link name="${name}_link">
+    <link name="${prefix}${name}_link">
       <visual>
         <geometry><cylinder radius="${wheel_r}" length="${wheel_w}"/></geometry>
@@ -62,10 +67,10 @@
   <xacro:wheel name="rear_left_wheel"   px="-${wheel_base_x}" py=" ${track}"/>
   <xacro:wheel name="rear_right_wheel"  px="-${wheel_base_x}" py="-${track}"/>
-  <joint name="lidar_joint" type="fixed">
-    <parent link="base_link"/>
-    <child  link="lidar_link"/>
+  <joint name="${prefix}lidar_joint" type="fixed">
+    <parent link="${prefix}base_link"/>
+    <child  link="${prefix}lidar_link"/>
     <origin xyz="0.28 0.0 ${base_z/2+0.04}" rpy="0 0 0"/>
   </joint>
-  <link name="lidar_link">
+  <link name="${prefix}lidar_link">
     <visual>
       <geometry><cylinder radius="0.045" length="0.07"/></geometry>
@@ -74,6 +79,6 @@
     <inertial><mass value="0.25"/><inertia ixx="0.0002" ixy="0" ixz="0" iyy="0.0002" iyz="0" izz="0.0003"/></inertial>
   </link>
-  <gazebo reference="lidar_link">
-    <sensor name="agv_lidar" type="ray">
+  <gazebo reference="${prefix}lidar_link">
+    <sensor name="${prefix}agv_lidar" type="ray">
       <always_on>true</always_on>
       <update_rate>10</update_rate>
@@ -99,43 +104,45 @@
         </noise>
       </ray>
-      <plugin name="agv_lidar_controller" filename="libgazebo_ros_ray_sensor.so">
+      <plugin name="${prefix}agv_lidar_controller" filename="libgazebo_ros_ray_sensor.so">
         <ros>
-          <namespace>/agv</namespace>
+          <namespace>/${robot_namespace}</namespace>
           <remapping>~/out:=scan</remapping>
         </ros>
         <output_type>sensor_msgs/LaserScan</output_type>
-        <frame_name>lidar_link</frame_name>
+        <frame_name>${prefix}lidar_link</frame_name>
       </plugin>
     </sensor>
   </gazebo>
-  <ros2_control name="agv_hardware" type="system">
-    <hardware><plugin>gazebo_ros2_control/GazeboSystem</plugin></hardware>
-    <joint name="front_left_wheel_joint">
-      <command_interface name="velocity"><param name="min">-3.0</param><param name="max">3.0</param></command_interface>
-      <state_interface name="position"/><state_interface name="velocity"/>
-    </joint>
-    <joint name="front_right_wheel_joint">
-      <command_interface name="velocity"><param name="min">-3.0</param><param name="max">3.0</param></command_interface>
-      <state_interface name="position"/><state_interface name="velocity"/>
-    </joint>
-    <joint name="rear_left_wheel_joint">
-      <command_interface name="velocity"><param name="min">-3.0</param><param name="max">3.0</param></command_interface>
-      <state_interface name="position"/><state_interface name="velocity"/>
-    </joint>
-    <joint name="rear_right_wheel_joint">
-      <command_interface name="velocity"><param name="min">-3.0</param><param name="max">3.0</param></command_interface>
-      <state_interface name="position"/><state_interface name="velocity"/>
-    </joint>
-  </ros2_control>
+  <xacro:if value="$(arg enable_ros2_control)">
+    <ros2_control name="${prefix}agv_hardware" type="system">
+      <hardware><plugin>gazebo_ros2_control/GazeboSystem</plugin></hardware>
+      <joint name="${prefix}front_left_wheel_joint">
+        <command_interface name="velocity"><param name="min">-3.0</param><param name="max">3.0</param></command_interface>
+        <state_interface name="position"/><state_interface name="velocity"/>
+      </joint>
+      <joint name="${prefix}front_right_wheel_joint">
+        <command_interface name="velocity"><param name="min">-3.0</param><param name="max">3.0</param></command_interface>
+        <state_interface name="position"/><state_interface name="velocity"/>
+      </joint>
+      <joint name="${prefix}rear_left_wheel_joint">
+        <command_interface name="velocity"><param name="min">-3.0</param><param name="max">3.0</param></command_interface>
+        <state_interface name="position"/><state_interface name="velocity"/>
+      </joint>
+      <joint name="${prefix}rear_right_wheel_joint">
+        <command_interface name="velocity"><param name="min">-3.0</param><param name="max">3.0</param></command_interface>
+        <state_interface name="position"/><state_interface name="velocity"/>
+      </joint>
+    </ros2_control>
+    <gazebo>
+      <plugin name="${prefix}gazebo_ros2_control" filename="libgazebo_ros2_control.so">
+        <parameters>$(find agv_description)/config/ros2_controllers.yaml</parameters>
+      </plugin>
+    </gazebo>
+  </xacro:if>
   <gazebo>
-    <plugin name="gazebo_ros2_control" filename="libgazebo_ros2_control.so">
-      <parameters>$(find agv_description)/config/ros2_controllers.yaml</parameters>
-    </plugin>
-  </gazebo>
-  <gazebo>
-    <plugin name="diff_drive_controller" filename="libgazebo_ros_diff_drive.so">
-      <ros><namespace>/agv</namespace></ros>
-      <left_joint>rear_left_wheel_joint</left_joint>
-      <right_joint>rear_right_wheel_joint</right_joint>
+    <plugin name="${prefix}diff_drive_controller" filename="libgazebo_ros_diff_drive.so">
+      <ros><namespace>/${robot_namespace}</namespace></ros>
+      <left_joint>${prefix}rear_left_wheel_joint</left_joint>
+      <right_joint>${prefix}rear_right_wheel_joint</right_joint>
       <wheel_separation>${track * 2}</wheel_separation>
       <wheel_diameter>${wheel_r * 2}</wheel_diameter>
@@ -143,10 +150,11 @@
       <publish_odom>true</publish_odom>
       <publish_odom_tf>true</publish_odom_tf>
-      <robot_base_frame>base_footprint</robot_base_frame>
+      <odometry_frame>${prefix}odom</odometry_frame>
+      <robot_base_frame>${prefix}base_footprint</robot_base_frame>
       <command_topic>cmd_vel</command_topic>
     </plugin>
   </gazebo>
   <xacro:macro name="wheel_physics" params="name mu">
-    <gazebo reference="${name}_link">
+    <gazebo reference="${prefix}${name}_link">
       <mu1>${mu}</mu1>
       <mu2>${mu}</mu2>
